File: final_schematics/fine_motor_control.kicad_sch (KiCad schematic)
At the start: 3 parts, among them J4 RJ9, U3 COM-09032

Commit message: Add flowcharts
Parts:
- added M1: Motor_DC, symbol Motor:Motor_DC
- added Q1: PN2222A, Package_TO_SOT_THT:TO-92_Inline, symbol Transistor_BJT:PN2222A
- added R1: 330, symbol Device:R_Small
Connections:
- net +5V: now also M1.1 (+)
- net GND: now also Q1.1 (E)
- net at A3.16 (D13): now also R1.1
- new net: Q1.2 (B), R1.2
- new net: M1.2 (-), Q1.3 (C)
